File: 1_energy-information-transduction/c_pd-starter/iv_pd-rpi/1.c.iv.2_rpi-pdwiringPi/digital_sensor.sch (EAGLE design)
At the start: 3 parts

Commit message: First full draft of 1.c.iv.2
Connections:
- removed net N$3: S1.S, U$1.11-GPIO17
- removed net N$4: R1.2, S1.S1
- new net GND: S1.P, U$1.6-GND
- net N$1: now also R1.2; no longer S1.P1
- net N$2: now also S1.S1, U$1.11-GPIO17
Other:
- moved on the sheet: R1, S1
Changed lines of the file:
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@@
 <part name="R1" library="adafruit" deviceset="R-US_" device="0207/12" value="10k"/>
 <part name="U$1" library="aliEagleLib" deviceset="RASPBERRY-PI" device=""/>
+<part name="SUPPLY1" library="supply2" deviceset="GND" device=""/>
+<part name="SUPPLY2" library="supply2" deviceset="GND" device=""/>
 </parts>
 <sheets>
@@
 </plain>
 <instances>
-<instance part="S1" gate="1" x="-35.56" y="-12.7" rot="R270"/>
-<instance part="R1" gate="G$1" x="35.56" y="22.86"/>
+<instance part="S1" gate="1" x="-48.26" y="20.32" rot="R270"/>
+<instance part="R1" gate="G$1" x="-33.02" y="38.1" rot="R90"/>
 <instance part="U$1" gate="G$1" x="5.08" y="0"/>
+<instance part="SUPPLY1" gate="GND" x="38.1" y="38.1"/>
+<instance part="SUPPLY2" gate="GND" x="-55.88" y="2.54"/>
 </instances>
 <busses>
@@
 <net name="N$1" class="0">
 <segment>
-<pinref part="S1" gate="1" pin="P1"/>
-<wire x1="-40.64" y1="-15.24" x2="-50.8" y2="-15.24" width="0.1524" layer="91"/>
-<wire x1="-50.8" y1="-15.24" x2="-50.8" y2="63.5" width="0.1524" layer="91"/>
-<wire x1="-50.8" y1="63.5" x2="30.48" y2="63.5" width="0.1524" layer="91"/>
+<wire x1="-33.02" y1="43.18" x2="-33.02" y2="63.5" width="0.1524" layer="91"/>
+<wire x1="-33.02" y1="63.5" x2="30.48" y2="63.5" width="0.1524" layer="91"/>
 <wire x1="30.48" y1="63.5" x2="30.48" y2="53.34" width="0.1524" layer="91"/>
 <pinref part="U$1" gate="G$1" pin="2-+5V"/>
 <wire x1="30.48" y1="53.34" x2="27.94" y2="53.34" width="0.1524" layer="91"/>
+<pinref part="R1" gate="G$1" pin="2"/>
 </segment>
 </net>
 <net name="N$2" class="0">
 <segment>
+<pinref part="S1" gate="1" pin="S1"/>
+<wire x1="-43.18" y1="17.78" x2="-33.02" y2="17.78" width="0.1524" layer="91"/>
+<pinref part="U$1" gate="G$1" pin="11-GPIO17"/>
+<wire x1="-20.32" y1="27.94" x2="-33.02" y2="27.94" width="0.1524" layer="91"/>
 <pinref part="R1" gate="G$1" pin="1"/>
-<wire x1="25.4" y1="22.86" x2="30.48" y2="22.86" width="0.1524" layer="91"/>
+<wire x1="-33.02" y1="27.94" x2="-33.02" y2="33.02" width="0.1524" layer="91"/>
+<wire x1="-33.02" y1="17.78" x2="-33.02" y2="27.94" width="0.1524" layer="91"/>
+<junction x="-33.02" y="27.94"/>
 </segment>
 </net>
-<net name="N$4" class="0">
+<net name="GND" class="0">
 <segment>
-<pinref part="S1" gate="1" pin="S1"/>
-<wire x1="-30.48" y1="-15.24" x2="-33.02" y2="-15.24" width="0.1524" layer="91"/>
-<wire x1="-30.48" y1="-15.24" x2="-25.4" y2="-15.24" width="0.1524" layer="91"/>
-<wire x1="-25.4" y1="-15.24" x2="-25.4" y2="-53.34" width="0.1524" layer="91"/>
-<junction x="-30.48" y="-15.24"/>
-<pinref part="R1" gate="G$1" pin="2"/>
-<wire x1="45.72" y1="22.86" x2="40.64" y2="22.86" width="0.1524" layer="91"/>
-<wire x1="-25.4" y1="-53.34" x2="45.72" y2="-53.34" width="0.1524" layer="91"/>
-<wire x1="45.72" y1="-53.34" x2="45.72" y2="22.86" width="0.1524" layer="91"/>
+<pinref part="SUPPLY2" gate="GND" pin="GND"/>
+<wire x1="-55.88" y1="5.08" x2="-55.88" y2="20.32" width="0.1524" layer="91"/>
+<pinref part="S1" gate="1" pin="P"/>
+<wire x1="-55.88" y1="20.32" x2="-53.34" y2="20.32" width="0.1524" layer="91"/>
+</segment>
+<segment>
+<pinref part="U$1" gate="G$1" pin="6-GND"/>
+<pinref part="SUPPLY1" gate="GND" pin="GND"/>
+<wire x1="27.94" y1="43.18" x2="38.1" y2="43.18" width="0.1524" layer="91"/>
+<wire x1="38.1" y1="43.18" x2="38.1" y2="40.64" width="0.1524" layer="91"/>
 </segment>
 </net>
-<net name="N$3" class="0">
-<segment>
-<pinref part="S1" gate="1" pin="S"/>
-<wire x1="-30.48" y1="-12.7" x2="-25.4" y2="-12.7" width="0.1524" layer="91"/>
-<wire x1="-25.4" y1="-12.7" x2="-25.4" y2="27.94" width="0.1524" layer="91"/>
-<pinref part="U$1" gate="G$1" pin="11-GPIO17"/>
-<wire x1="-25.4" y1="27.94" x2="-20.32" y2="27.94" width="0.1524" layer="91"/>
-</segment>
-</net>

Commit message: Changing Raspberry Pi GPIO circuit to use 3.3V.
Connections:
- net N$1: now also U$1.1-+3V3; no longer U$1.2-+5V
Changed lines of the file:
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@@
 <net name="N$1" class="0">
 <segment>
-<wire x1="-33.02" y1="43.18" x2="-33.02" y2="63.5" width="0.1524" layer="91"/>
-<wire x1="-33.02" y1="63.5" x2="30.48" y2="63.5" width="0.1524" layer="91"/>
-<wire x1="30.48" y1="63.5" x2="30.48" y2="53.34" width="0.1524" layer="91"/>
-<pinref part="U$1" gate="G$1" pin="2-+5V"/>
-<wire x1="30.48" y1="53.34" x2="27.94" y2="53.34" width="0.1524" layer="91"/>
+<wire x1="-33.02" y1="43.18" x2="-33.02" y2="53.34" width="0.1524" layer="91"/>
 <pinref part="R1" gate="G$1" pin="2"/>
+<pinref part="U$1" gate="G$1" pin="1-+3V3"/>
+<wire x1="-33.02" y1="53.34" x2="-20.32" y2="53.34" width="0.1524" layer="91"/>
 </segment>
 </net>
